File: THAT1510_xx12/THAT15xx_DSheet.brd (EAGLE design)
At the start: 24.1 x 22.1 mm, 19 parts, among them U1 THAT1512PO8-U

Commit message: Added THAT15xx
Added THAT15xx
Parts:
- GAIN: value B10k -> B1K
Changed lines of the file:
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@@
 <layer number="23" name="tOrigins" color="15" fill="1" visible="yes" active="yes"/>
 <layer number="24" name="bOrigins" color="15" fill="1" visible="yes" active="yes"/>
-<layer number="25" name="tNames" color="7" fill="1" visible="yes" active="yes"/>
-<layer number="26" name="bNames" color="7" fill="1" visible="yes" active="yes"/>
+<layer number="25" name="tNames" color="7" fill="1" visible="no" active="yes"/>
+<layer number="26" name="bNames" color="7" fill="1" visible="no" active="yes"/>
 <layer number="27" name="tValues" color="7" fill="1" visible="no" active="yes"/>
 <layer number="28" name="bValues" color="7" fill="1" visible="no" active="yes"/>
@@
 <layer number="50" name="dxf" color="7" fill="1" visible="no" active="no"/>
 <layer number="51" name="tDocu" color="6" fill="1" visible="yes" active="yes"/>
-<layer number="52" name="bDocu" color="7" fill="1" visible="yes" active="yes"/>
+<layer number="52" name="bDocu" color="7" fill="1" visible="no" active="yes"/>
 <layer number="53" name="tGND_GNDA" color="7" fill="1" visible="no" active="no"/>
 <layer number="54" name="bGND_GNDA" color="7" fill="1" visible="no" active="no"/>
@@
 <attribute name="VALUE" x="20.087" y="13.91" size="0.7" layer="27" rot="R90"/>
 </element>
-<element name="GAIN" library="MusicThingModular" package="9MM_SNAP-IN_POT" value="B10k" x="17.653" y="8.382" smashed="yes" rot="MR0">
+<element name="GAIN" library="MusicThingModular" package="9MM_SNAP-IN_POT" value="B1K" x="17.653" y="8.382" smashed="yes" rot="MR0">
 <attribute name="NAME" x="19.558" y="14.224" size="0.7" layer="26" rot="MR0"/>
 <attribute name="VALUE" x="21.463" y="4.572" size="0.7" layer="28" rot="MR0"/>
