File: THAT1510_xx12/THAT15xx_DSheet.sch (EAGLE design)
At the start: 19 parts, among them U1 THAT1512PO8-U

Commit message: Added THAT15xx
Added THAT15xx
Parts:
- GAIN: value B10k -> B1K
Other:
- note added: "Filter varies with gain setting. Datasheet recommends 3300uF."
- note removed: "Varies with Gain Setting. Safe bet? 6800uF for the 1512 & 3300uF for the 1510. Way we'll play it? 470uF probs..."
Changed lines of the file:
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@@
 <part name="GND7" library="supply pins" deviceset="GND" device=""/>
 <part name="GND8" library="supply pins" deviceset="GND" device=""/>
-<part name="GAIN" library="MusicThingModular" deviceset="9MM_SNAP-IN_POT_CHASSIS" device="" value="B10k"/>
+<part name="GAIN" library="MusicThingModular" deviceset="9MM_SNAP-IN_POT_CHASSIS" device="" value="B1K"/>
 <part name="C6" library="MusicThingModular" deviceset="CAP_SMD+THRU" device="PAN_C" value="Cg"/>
 <part name="GND9" library="supply pins" deviceset="GND" device=""/>
@@
 <sheet>
 <plain>
-<text x="34.036" y="58.928" size="1.27" layer="97">Varies with Gain Setting.
-Safe bet?
-6800uF for the 1512
-&amp; 3300uF for the 1510.
-Way we'll play it?
-470uF probs...</text>
+<text x="34.036" y="58.928" size="1.27" layer="97">Filter varies with
+gain setting.
+Datasheet recommends
+3300uF.</text>
 </plain>
 <instances>
